Commit message: Use portable package:// mesh paths in the DynaArm URDF.
Isaac Lab 2.3 still needs absolute mesh files, so spawn rewrites those
URIs against the duatic_dynaarm submodule at USD conversion.

File: source/isaaclab_hiveboard/isaaclab_hiveboard/assets/anymal/urdf/dynaarm.urdf (robot description, URDF)
Before this commit: robot dynaarm, 11 links, 10 joints
Links:
- link dynaarm_base: geometry collision cylinder length=0.1 radius=0.05; visual mesh filename=package://duatic_dynaarm_description/meshes/corydoras12/bas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 scale=1.0 1.0 1.0
- link dynaarm_elbow: geometry collision cylinder length=0.2 radius=0.065; visual mesh filename=package://duatic_dynaarm_description/meshes/corydoras12/elb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 scale=1.0 1.0 1.0
- link dynaarm_forearm: geometry collision cylinder length=0.4 radius=0.04; visual mesh filename=package://duatic_dynaarm_description/meshes/corydoras12/for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 scale=1.0 1.0 1.0
- link dynaarm_shoulder: geometry collision cylinder length=0.25 radius=0.06; visual mesh filename=package://duatic_dynaarm_description/meshes/corydoras12/sho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 scale=1.0 1.0 1.0
- link dynaarm_upperarm: geometry collision cylinder length=0.4 radius=0.05; visual mesh filename=package://duatic_dynaarm_description/meshes/corydoras12/upp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 scale=1.0 1.0 1.0
- link dynaarm_wrist_1: geometry collision cylinder length=0.125 radius=0.05; visual mesh filename=package://duatic_dynaarm_description/meshes/corydoras12/wri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 scale=1.0 1.0 1.0
- link dynaarm_wrist_2: geometry collision cylinder length=0.09 radius=0.052; visual mesh filename=package://duatic_dynaarm_description/meshes/corydoras12/wri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 scale=1.0 1.0 1.0
