Commit message: astra changes

File: source/isaaclab_hiveboard/isaaclab_hiveboard/assets/spot/spot_with_arm.urdf (robot description, URDF)
Before this commit: robot spot_with_arm, 25 links, 24 joints
Links:
- link arm_link_jaw: mass None -> 1e-6
- link fl_foot: mass None -> 1e-6
- link fr_foot: mass None -> 1e-6
- link hl_foot: mass None -> 1e-6
- link hr_foot: mass None -> 1e-6
