Commit message: Guide the drawer by shaft contact instead of a prismatic joint.
The box is a free body and the housing stays fixed. A straight pull stops on the lip; open is still 20 mm of forward travel inside the slot.

File: source/isaaclab_hiveboard/isaaclab_hiveboard/assets/hiveboard/drawer/Drawer_Assembly.urdf (robot description, URDF)
Before this commit: robot Drawer_Assembly, 2 links, 1 joints
Links:
- link base: geometry collision box size=0.013 0.042 0.070; collision box size=0.013 0.042 0.070
- link drawer: geometry collision box size=0.010 0.030 0.010; collision cylinder length=0.046 radius=0.004
Joints:
- removed joint PrismaticJoint
- added joint float: type floating, parent base, child drawer, origin xyz=0 0 0 rpy=0 0 0

Commit message: Fix drawer contact physics and complete removal sequences

File: source/isaaclab_hiveboard/isaaclab_hiveboard/assets/hiveboard/drawer/Drawer_Assembly.urdf (robot description, URDF)
Before this commit: robot Drawer_Assembly, 2 links, 1 joints
Links:
- link base: geometry collision box size=0.0024554408 0.0018857142 0.0067922194; collision box size=0.0024554408 0.0018857142 0.0067922194
- link drawer: geometry collision box size=0.010 0.030 0.010; collision box size=0.033 0.002 0.04355
